Commit message: somlify botanbot meshes

File: botanbot_description/urdf/botanbot.urdf (robot description, URDF)
Before this commit: robot botanbot, 21 links, 20 joints
Links:
- link base_link: geometry collision mesh filename=package://botanbot_description/meshes/base_simplified.stl; visual mesh filename=package://botanbot_description/meshes/base_simplified.stl
- link front_left_wheel: geometry collision mesh filename=package://botanbot_description/meshes/wheel_simplified.stl scale=1 1 1; visual mesh filename=package://botanbot_description/meshes/wheel_simplified.stl scale=1 1 1
- link front_right_wheel: geometry collision mesh filename=package://botanbot_description/meshes/wheel_simplified.stl scale=1 1 1; visual mesh filename=package://botanbot_description/meshes/wheel_simplified.stl scale=1 1 1
- link rear_left_wheel: geometry collision mesh filename=package://botanbot_description/meshes/wheel_simplified.stl scale=1 1 1; visual mesh filename=package://botanbot_description/meshes/wheel_simplified.stl scale=1 1 1
- link rear_right_wheel: geometry collision mesh filename=package://botanbot_description/meshes/wheel_simplified.stl scale=1 1 1; visual mesh filename=package://botanbot_description/meshes/wheel_simplified.stl scale=1 1 1
- link steering_wheel: geometry collision mesh filename=package://botanbot_description/meshes/wheel_simplified.stl scale=0.5 0.5 1; visual mesh filename=package://botanbot_description/meshes/wheel_simplified.stl scale=0.5 0.5 1

Commit message: integrate joystick to botanbot

File: botanbot_description/urdf/botanbot.urdf (robot description, URDF)
Before this commit: robot botanbot, 21 links, 20 joints
Links:
- removed link gps
- added link gps_link; collision mesh filename=package://botanbot_description/meshes/gps.stl scale=0.0005 0.0005 0.001; visual mesh filename=package://botanbot_description/meshes/gps.stl scale=0.0005 0.0005 0.001
Joints:
- joint gps_joint: child gps -> gps_link

Commit message: clash vox_nav and navigation2

File: botanbot_description/urdf/botanbot.urdf (robot description, URDF)
Before this commit: robot botanbot, 21 links, 20 joints
Links:
- removed link velodyne_link
- added link lidar_data_link; collision mesh filename=package://botanbot_description/meshes/lidar.stl scale=0.001 0.001 0.001; visual mesh filename=package://botanbot_description/meshes/lidar.stl scale=0.001 0.001 0.001
Joints:
- joint velodyne_joint: child velodyne_link -> lidar_data_link
